Commit message: Física de la rueda castor OK. Se añadió plugin de movimiento.

File: install/modelo_robot/share/modelo_robot/urdf/Seguidor_linea_robot.urdf (robot description, URDF)
Before this commit: robot mobile_robot, 5 links, 4 joints
Links:
- link Base_castor_link: mass 0.1 -> 0.5

Commit message: Added LaserScan

File: install/modelo_robot/share/modelo_robot/urdf/Seguidor_linea_robot.urdf (robot description, URDF)
Before this commit: robot mobile_robot, 5 links, 4 joints
Links:
- added link Lidar_link, mass 0.01; collision cylinder length=0.02 radius=0.01; visual cylinder length=0.04 radius=0.01
Joints:
- added joint Lidar_joint: type fixed, parent base_link, child Lidar_link, origin xyz=0.0 0.0 0.02 rpy=0 -0.05 0, axis 1 0 0

Commit message: Added Lidar and IMU sensors

File: install/modelo_robot/share/modelo_robot/urdf/Seguidor_linea_robot.urdf (robot description, URDF)
Before this commit: robot mobile_robot, 6 links, 5 joints
Links:
- added link imu_link
- link Lidar_link: geometry collision cylinder length=0.05 radius=0.01; visual cylinder length=0.05 radius=0.01
Joints:
- added joint imu_joint: type fixed, parent base_link, child imu_link, origin xyz=0.0 0 0.0 rpy=0 0 0, axis 1 0 0
- joint Lidar_joint: origin xyz=0.0 0.0 0.02 rpy=0 -0.05 0 -> xyz=0.0 0 0.0 rpy=0 -0.08 0

Commit message: Added slam toolbox node for mapping

File: install/modelo_robot/share/modelo_robot/urdf/Seguidor_linea_robot.urdf (robot description, URDF)
Before this commit: robot mobile_robot, 7 links, 6 joints
Links:
- added link base_link_ground
Joints:
- added joint ground_base_joint: type fixed, parent base_link, child base_link_ground, origin xyz=0.0 0.0 -0.05 rpy=0.0 0.0 0.0

Commit message: Slam mapper + fixed tfs

File: install/modelo_robot/share/modelo_robot/urdf/Seguidor_linea_robot.urdf (robot description, URDF)
Before this commit: robot mobile_robot, 8 links, 7 joints
Joints:
- joint Lidar_joint: origin xyz=0.0 0 0.0 rpy=0 -0.08 0 -> xyz=0.0 0 0.02 rpy=0 -0.087 0
- joint ground_base_joint: child base_link_ground -> base_link; origin xyz=0.0 0.0 -0.05 rpy=0.0 0.0 0.0 -> xyz=0.0 0.0 0.05 rpy=0.0 0.0 0.0; parent base_link -> base_link_ground
