Commit message: Added autonomous navigation stack and lab map

File: src/modelo_robot/urdf/Seguidor_linea_robot.urdf (robot description, URDF)
Before this commit: robot mobile_robot, 8 links, 7 joints
Links:
- added link camera_link, mass 0.03; collision box size=0.02 0.02 0.02; visual box size=0.02 0.02 0.02
Joints:
- added joint camera_joint: type fixed, parent base_link, child camera_link, origin xyz=0.05 0.0 0.01 rpy=0.0 0.0 0.0
- joint imu_joint: origin xyz=0.0 0 0.0 rpy=0 0 0 -> xyz=0.0 0 0.0 rpy=0 -0.07 0

Commit message: Merged dev with main

File: src/modelo_robot/urdf/Seguidor_linea_robot.urdf (robot description, URDF)
Before this commit: robot mobile_robot, 5 links, 4 joints
Links:
- added link Lidar_link, mass 0.01; collision cylinder length=0.05 radius=0.01; visual cylinder length=0.05 radius=0.01
- added link base_link_ground
- added link camera_link, mass 0.03; collision box size=0.02 0.02 0.02; visual box size=0.02 0.02 0.02
- added link imu_link
- link Base_castor_link: mass 0.1 -> 0.5; geometry collision mesh filename=package://modelo_robot/meshes/Base_castor_link.STL; visual mesh filename=package://modelo_robot/meshes/Base_castor_link.STL
- link Rueda_castor_link: geometry collision mesh filename=package://modelo_robot/meshes/Rueda_castor_link.STL; visual mesh filename=package://modelo_robot/meshes/Rueda_castor_link.STL
- link Rueda_derecha_link: geometry collision mesh filename=package://modelo_robot/meshes/Rueda_derecha_link.STL; visual mesh filename=package://modelo_robot/meshes/Rueda_derecha_link.STL
- link Rueda_izquierda_link: geometry collision mesh filename=package://modelo_robot/meshes/Rueda_izquierda_link.STL; visual mesh filename=package://modelo_robot/meshes/Rueda_izquierda_link.STL
- link base_link: geometry collision mesh filename=package://modelo_robot/meshes/base_link.STL; visual mesh filename=package://modelo_robot/meshes/base_link.STL
Joints:
- added joint Lidar_joint: type fixed, parent base_link, child Lidar_link, origin xyz=0.0 0 0.02 rpy=0 -0.087 0, axis 1 0 0
- added joint camera_joint: type fixed, parent base_link, child camera_link, origin xyz=0.05 0.0 0.01 rpy=0.0 0.0 0.0
- added joint ground_base_joint: type fixed, parent base_link_ground, child base_link, origin xyz=0.0 0.0 0.05 rpy=0.0 0.0 0.0
- added joint imu_joint: type fixed, parent base_link, child imu_link, origin xyz=0.0 0 0.0 rpy=0 -0.07 0, axis 1 0 0
